File: AccessControlBoard/AccessControlBoard.sch (EAGLE design)
At the start: 9 parts, among them J1 4p-2.54, X1 1751248

Commit message: update
Parts:
- removed J1: 4p-2.54, Seeed-Connector:DIP-BLACK-FEMALE-HEADER-VERT(4P-2.54)
- added C1, C2: 22uF, rcl:C-EUC0805K
- added C3, C4: 100nF, rcl:C-EUC0603K
- added CN1: 6p-2.54, Seeed-Connector:DIP-BLACK-FEMALE-HEADER-VERT(6P-2.54)
- added D1: 1N4007, Seeed-Diode:DIODE-GEN-PURPOSE-1KV-1A(DO-214AC)
- added Q1: AO3400, Seeed-Transistor:SMD-MOSFET-N-CH-60V-300MA-LOGIC-LEVEL-FET-2N7002(SOT-23)
- added R1, R2, R3, R7: 10k, resistor:R-US_R0603
- added R4: S07K17, varistor:S07K17
- added R5: 2ohm, resistor:R-US_R0603
- added R6: 3.3k, resistor:R-US_R0603
Connections:
- new net ADC: U1.ADC
- new net EN: C4.2, R7.2, U1.CH_PD
- new net GPIO0: C4.1, CN1.6, R2.2, U1.GPIO0
- new net GPIO2: R3.2, U1.GPIO2
- new net N$5: C1.1, D1.-, R5.2, U$1.COIL0
- new net N$8: D1.+, Q1.D, U$1.COIL1
- new net RLY: Q1.G, U1.GPIO16
- new net RX: CN1.4, U1.RX
- new net SW: R6.2, S1.S, U1.GPIO5, X1-2.K
- new net TX: CN1.5, U1.TX
- net +3V3: now also C2.2, C3.2, R2.1, R3.1, R5.1, R6.1, R7.1
- net CS: now also R1.2, U1.GPIO15
- net GND: now also C1.2, C2.1, C3.1, CN1.1, Q1.S, R1.1, S1.P; no longer J1.P$1
- net IRQ: now also U1.GPIO4
- net MISO: now also U1.GPIO12
- net MOSI: now also U1.GPIO13
- net N$2: now also R4.2
- net N$3: now also R4.1
- net RST: now also U1.RESET
- net SCK: now also U1.GPIO14
Other:
- note added: "Button/external contact"
- note added: "ESP module"
- note added: "FTDI programming"
- note added: "MFRC522 board connector"
- note added: "Note: RST pulled up internally, also by RFID board via 1k resistor"
- note added: "Power supply"
- note added: "Relay"
- moved on the sheet: F1, HLK1, JP1, S1, U$1, U1, X1-1, X2-1, X2-2, X2-3

Commit message: board release candidate
Parts:
- added C5: (no value), rcl:C-EU102-064X133
- added C6: 22uF, rcl:C-EUC0805K
- added U$2: L, adafruit:L
- R4: value S07K17 -> S07K250; device varistor:S07K17 -> varistor:S07K250
Connections:
- new net N$6: HLK1.AC2, U$2.1
- net +3V3: now also C6.2, CN1.3
- net GND: now also C6.1
- net N$2: now also C5.1
- net N$3: now also C5.2, U$2.2; no longer HLK1.AC2
Other:
- moved on the sheet: F1, R4
Changed lines of the file:
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@@
 <part name="R6" library="resistor" library_urn="urn:adsk.eagle:library:348" deviceset="R-US_" device="R0603" package3d_urn="urn:adsk.eagle:package:26057/1" value="3.3k"/>
 <part name="CN1" library="Seeed-Connector" library_urn="urn:adsk.eagle:library:478" deviceset="DIP-BLACK-FEMALE-HEADER-VERT(6P-2.54)" device="" package3d_urn="urn:adsk.eagle:package:33114/1" value="6p-2.54"/>
-<part name="R4" library="varistor" library_urn="urn:adsk.eagle:library:410" deviceset="S07K17" device="" package3d_urn="urn:adsk.eagle:package:30546/1"/>
+<part name="R4" library="varistor" library_urn="urn:adsk.eagle:library:410" deviceset="S07K250" device="" package3d_urn="urn:adsk.eagle:package:30540/1"/>
 <part name="C4" library="rcl" library_urn="urn:adsk.eagle:library:334" deviceset="C-EU" device="C0603K" package3d_urn="urn:adsk.eagle:package:23680/2" value="100nF"/>
 <part name="R7" library="resistor" library_urn="urn:adsk.eagle:library:348" deviceset="R-US_" device="R0603" package3d_urn="urn:adsk.eagle:package:26057/1" value="10k"/>
 <part name="+3V6" library="supply1" library_urn="urn:adsk.eagle:library:371" deviceset="+3V3" device=""/>
+<part name="C5" library="rcl" library_urn="urn:adsk.eagle:library:334" deviceset="C-EU" device="102-064X133" package3d_urn="urn:adsk.eagle:package:23653/1"/>
+<part name="U$2" library="adafruit" library_urn="urn:adsk.eagle:library:420" deviceset="L" device=""/>
+<part name="+3V9" library="supply1" library_urn="urn:adsk.eagle:library:371" deviceset="+3V3" device=""/>
+<part name="C6" library="rcl" library_urn="urn:adsk.eagle:library:334" deviceset="C-EU" device="C0805K" package3d_urn="urn:adsk.eagle:package:23681/2" value="22uF"/>
 </parts>
 <sheets>
@@
 <instance part="X2" gate="-2" x="20.32" y="30.48"/>
 <instance part="X2" gate="-3" x="20.32" y="60.96"/>
-<instance part="F1" gate="G$1" x="35.56" y="15.24"/>
+<instance part="F1" gate="G$1" x="22.86" y="10.16"/>
 <instance part="JP1" gate="G$1" x="129.54" y="105.41" rot="R180"/>
 <instance part="U1" gate="G$1" x="48.26" y="147.32"/>
@@
 <instance part="R6" gate="G$1" x="208.28" y="119.38" rot="R270"/>
 <instance part="CN1" gate="G$1" x="134.62" y="143.51" rot="R180"/>
-<instance part="R4" gate="G$1" x="43.18" y="20.32" rot="R90"/>
+<instance part="R4" gate="G$1" x="35.56" y="17.78" rot="R90"/>
 <instance part="C4" gate="G$1" x="154.94" y="154.94" rot="R90"/>
 <instance part="R7" gate="G$1" x="167.64" y="157.48" rot="R270"/>
 <instance part="+3V6" gate="G$1" x="167.64" y="167.64"/>
+<instance part="C5" gate="G$1" x="30.48" y="15.24"/>
+<instance part="U$2" gate="G$1" x="43.18" y="10.16" rot="R270"/>
+<instance part="+3V9" gate="G$1" x="160.02" y="144.78"/>
+<instance part="C6" gate="G$1" x="121.92" y="22.86"/>
 </instances>
 <busses>
@@
 <net name="N$2" class="0">
 <segment>
-<wire x1="25.4" y1="35.56" x2="40.64" y2="35.56" width="0.1524" layer="91"/>
-<wire x1="40.64" y1="35.56" x2="43.18" y2="25.4" width="0.1524" layer="91"/>
+<wire x1="25.4" y1="35.56" x2="35.56" y2="35.56" width="0.1524" layer="91"/>
+<wire x1="35.56" y1="35.56" x2="35.56" y2="22.86" width="0.1524" layer="91"/>
 <pinref part="HLK1" gate="G$1" pin="AC1"/>
-<wire x1="43.18" y1="25.4" x2="50.8" y2="22.86" width="0.1524" layer="91"/>
+<wire x1="35.56" y1="22.86" x2="50.8" y2="22.86" width="0.1524" layer="91"/>
 <pinref part="U$1" gate="G$1" pin="SWCOMMON"/>
-<wire x1="40.64" y1="35.56" x2="40.64" y2="55.88" width="0.1524" layer="91"/>
-<wire x1="40.64" y1="55.88" x2="53.34" y2="55.88" width="0.1524" layer="91"/>
-<junction x="40.64" y="35.56"/>
+<wire x1="35.56" y1="35.56" x2="35.56" y2="55.88" width="0.1524" layer="91"/>
+<wire x1="35.56" y1="55.88" x2="53.34" y2="55.88" width="0.1524" layer="91"/>
+<junction x="35.56" y="35.56"/>
 <pinref part="X2" gate="-1" pin="KL"/>
 <pinref part="R4" gate="G$1" pin="2"/>
-<junction x="43.18" y="25.4"/>
+<junction x="35.56" y="22.86"/>
+<pinref part="C5" gate="G$1" pin="1"/>
+<wire x1="30.48" y1="17.78" x2="30.48" y2="22.86" width="0.1524" layer="91"/>
+<wire x1="30.48" y1="22.86" x2="35.56" y2="22.86" width="0.1524" layer="91"/>
 </segment>
 </net>
 <net name="N$3" class="0">
 <segment>
-<pinref part="HLK1" gate="G$1" pin="AC2"/>
-<wire x1="40.64" y1="15.24" x2="43.18" y2="15.24" width="0.1524" layer="91"/>
+<wire x1="27.94" y1="10.16" x2="30.48" y2="10.16" width="0.1524" layer="91"/>
 <pinref part="F1" gate="G$1" pin="2"/>
 <pinref part="R4" gate="G$1" pin="1"/>
-<wire x1="43.18" y1="15.24" x2="50.8" y2="17.78" width="0.1524" layer="91"/>
-<junction x="43.18" y="15.24"/>
+<pinref part="U$2" gate="G$1" pin="2"/>
+<junction x="35.56" y="10.16"/>
+<wire x1="30.48" y1="10.16" x2="35.56" y2="10.16" width="0.1524" layer="91"/>
+<wire x1="35.56" y1="10.16" x2="35.56" y2="12.7" width="0.1524" layer="91"/>
+<pinref part="C5" gate="G$1" pin="2"/>
+<junction x="30.48" y="10.16"/>
 </segment>
 </net>
@@
 <segment>
 <wire x1="25.4" y1="30.48" x2="25.4" y2="15.24" width="0.1524" layer="91"/>
-<wire x1="25.4" y1="15.24" x2="30.48" y2="15.24" width="0.1524" layer="91"/>
+<wire x1="25.4" y1="15.24" x2="17.78" y2="10.16" width="0.1524" layer="91"/>
 <pinref part="F1" gate="G$1" pin="1"/>
 <pinref part="X2" gate="-2" pin="KL"/>
@@
 <pinref part="HLK1" gate="G$1" pin="-VO"/>
 <pinref part="GND1" gate="1" pin="GND"/>
-<wire x1="129.54" y1="27.94" x2="111.76" y2="27.94" width="0.1524" layer="91"/>
+<wire x1="129.54" y1="27.94" x2="121.92" y2="27.94" width="0.1524" layer="91"/>
 <pinref part="C2" gate="G$1" pin="1"/>
+<wire x1="121.92" y1="27.94" x2="111.76" y2="27.94" width="0.1524" layer="91"/>
 <wire x1="111.76" y1="27.94" x2="99.06" y2="27.94" width="0.1524" layer="91"/>
 <wire x1="99.06" y1="27.94" x2="91.44" y2="27.94" width="0.1524" layer="91"/>
@@
 <wire x1="111.76" y1="25.4" x2="111.76" y2="27.94" width="0.1524" layer="91"/>
 <junction x="111.76" y="27.94"/>
+<pinref part="C6" gate="G$1" pin="1"/>
+<wire x1="121.92" y1="25.4" x2="121.92" y2="27.94" width="0.1524" layer="91"/>
+<junction x="121.92" y="27.94"/>
 </segment>
 <segment>
@@
 <pinref part="HLK1" gate="G$1" pin="+VO"/>
 <pinref part="+3V1" gate="G$1" pin="+3V3"/>
-<wire x1="129.54" y1="12.7" x2="111.76" y2="12.7" width="0.1524" layer="91"/>
+<wire x1="129.54" y1="12.7" x2="121.92" y2="12.7" width="0.1524" layer="91"/>
 <pinref part="C2" gate="G$1" pin="2"/>
+<wire x1="121.92" y1="12.7" x2="111.76" y2="12.7" width="0.1524" layer="91"/>
 <wire x1="111.76" y1="12.7" x2="99.06" y2="12.7" width="0.1524" layer="91"/>
 <wire x1="99.06" y1="12.7" x2="91.44" y2="12.7" width="0.1524" layer="91"/>
@@
 <wire x1="111.76" y1="17.78" x2="111.76" y2="12.7" width="0.1524" layer="91"/>
 <junction x="111.76" y="12.7"/>
+<pinref part="C6" gate="G$1" pin="2"/>
+<wire x1="121.92" y1="17.78" x2="121.92" y2="12.7" width="0.1524" layer="91"/>
+<junction x="121.92" y="12.7"/>
 </segment>
 <segment>
@@
 <pinref part="+3V6" gate="G$1" pin="+3V3"/>
 <wire x1="167.64" y1="162.56" x2="167.64" y2="165.1" width="0.1524" layer="91"/>
+</segment>
+<segment>
+<pinref part="CN1" gate="G$1" pin="3"/>
+<wire x1="142.24" y1="142.24" x2="147.32" y2="142.24" width="0.1524" layer="91"/>
+<wire x1="147.32" y1="142.24" x2="147.32" y2="139.7" width="0.1524" layer="91"/>
+<pinref part="+3V9" gate="G$1" pin="+3V3"/>
+<wire x1="147.32" y1="139.7" x2="160.02" y2="139.7" width="0.1524" layer="91"/>
+<wire x1="160.02" y1="139.7" x2="160.02" y2="142.24" width="0.1524" layer="91"/>
 </segment>
 </net>
@@
 </segment>
 </net>
+<net name="N$6" class="0">
+<segment>
+<pinref part="HLK1" gate="G$1" pin="AC2"/>
+<pinref part="U$2" gate="G$1" pin="1"/>
+<wire x1="50.8" y1="10.16" x2="50.8" y2="17.78" width="0.1524" layer="91"/>
+</segment>
+</net>
