File: AccessControlBoard/AccessControlBoard.brd (EAGLE design)
At the start: 43.2 x 62.2 mm, 9 parts, among them J1 4p-2.54, X1 1751248

Commit message: update
Parts:
- removed J1: 4p-2.54, Seeed-Connector:H4-2.54
- added C1, C2: 22uF, rcl:C0805K
- added C3, C4: 100nF, rcl:C0603K
- added CN1: 6p-2.54, Seeed-Connector:H6-2.54
- added D1: 1N4007, Seeed-Diode:DO-214AC
- added Q1: AO3400, Seeed-Transistor:SOT-23
- added R1, R2, R3, R7: 10k, resistor:R0603
- added R4: S07K17, varistor:S07K17
- added R5: 2ohm, resistor:R0603
- added R6: 3.3k, resistor:R0603
- moved S1 24.7 mm to (3.81, 5.08), turned to 270 degrees
- moved F1 3.88 mm to (1.59, 19.7)
- moved U$1 1.62 mm to (9.84, 44.8)
Connections:
- new net ADC: U1.ADC
- new net EN: C4.2, R7.2, U1.CH_PD
- new net GPIO0: C4.1, CN1.6, R2.2, U1.GPIO0
- new net GPIO2: R3.2, U1.GPIO2
- new net N$5: C1.1, D1.2, R5.2, U$1.COIL0
- new net N$8: D1.1, Q1.3, U$1.COIL1
- new net RLY: Q1.1, U1.GPIO16
- new net RX: CN1.4, U1.RXD0
- new net SW: R6.2, S1.2, U1.GPIO5, X1.2
- new net TX: CN1.5, U1.TXD0
- net +3V3: now also C2.2, C3.2, R2.1, R3.1, R5.1, R6.1, R7.1
- net CS: now also R1.2, U1.GPIO15
- net GND: now also C1.2, C2.1, C3.1, CN1.1, Q1.2, R1.1, S1.1; no longer J1.1
- net IRQ: now also U1.GPIO4
- net MISO: now also U1.GPIO12
- net MOSI: now also U1.GPIO13
- net N$2: now also R4.2
- net N$3: now also R4.1
- net RST: now also U1.RESET
- net SCK: now also U1.GPIO14
Routing:
- net SW: track 0.00 -> 94.5 mm, vias 0 -> 3
- net +3V3: track 0.00 -> 74.6 mm
- net IRQ: track 0.00 -> 73.5 mm, vias 0 -> 1
- net CS: track 0.00 -> 63.5 mm, vias 0 -> 1
- net SCK: track 0.00 -> 51.2 mm, vias 0 -> 1
- net MISO: track 0.00 -> 49.8 mm, vias 0 -> 1
- net MOSI: track 0.00 -> 46.8 mm, vias 0 -> 1
- net RX: track 0.00 -> 33.6 mm, vias 0 -> 1
- net TX: track 0.00 -> 31.5 mm, vias 0 -> 1
- net N$5: track 0.00 -> 30.2 mm
- net RLY: track 0.00 -> 27.3 mm, vias 0 -> 2
- net GPIO0: track 0.00 -> 27.1 mm
- net N$2: track 49.5 -> 74.9 mm
- net EN: track 0.00 -> 23.2 mm
- net GPIO2: track 0.00 -> 14.7 mm
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Other:
- outline, holes or cut-outs redrawn
- board text added: "F125mA"
- board text added: "RESERVED AREA FOR FILTER"
- board text added: "~"

Commit message: board release candidate
Parts:
- added C5: (no value), rcl:C102-064X133
- added C6: 22uF, rcl:C0805K
- added U$2: L, adafruit:6000
- R4: value S07K17 -> S07K250; device varistor:S07K17 -> varistor:S07K250
- moved F1 16.2 mm to (6.03, 35.2), turned to 0 degrees
- moved R4 12.6 mm to (9.84, 28.9), turned to 180 degrees
- moved C3 4.97 mm to (26.4, 35.9), turned to 180 degrees
- moved C1 3.86 mm to (22.2, 35.6), turned to 90 degrees
- moved R5 2.62 mm to (22.2, 30.8), turned to 90 degrees
- moved CN1 1.42 mm to (34.3, 25.7)
- moved C4 1.35 mm to (34.3, 35.6)
- moved Q1 1.35 mm to (18.4, 26.4), turned to 0 degrees
- moved R7 1.27 mm to (31.1, 31.4)
- moved D1 1.14 mm to (18.4, 32.4), turned to 90 degrees
- moved R6 0.95 mm to (34.3, 31.4)
- moved HLK1 0.71 mm to (26.0, 13.7)
- moved R2 0.64 mm to (37.5, 31.4)
- moved U1 0.63 mm to (33.0, 47.6)
- moved R3 0.32 mm to (40.6, 31.4)
Connections:
- new net N$6: HLK1.P$2, U$2.1
- net +3V3: now also C6.2, CN1.3
- net GND: now also C6.1
- net N$2: now also C5.1
- net N$3: now also C5.2, U$2.2; no longer HLK1.P$2
Routing:
- net N$3: track 10.5 -> 30.0 mm
- net IRQ: track 73.5 -> 58.8 mm
- net N$4: track 37.6 -> 25.3 mm
- net SW: track 94.5 -> 103.0 mm, vias 3 -> 2
- net N$6: track 0.00 -> 6.99 mm
- net N$2: track 74.9 -> 80.7 mm
- net RX: track 33.6 -> 29.2 mm
- net +3V3: track 74.6 -> 71.6 mm
- net GPIO0: track 27.1 -> 29.2 mm
- net N$5: track 30.2 -> 28.4 mm
- net N$8: track 12.0 -> 13.5 mm
- net GPIO2: track 14.7 -> 16.0 mm
- net SCK: track 51.2 -> 50.5 mm
- net RLY: track 27.3 -> 27.8 mm
Other:
- outline, holes or cut-outs redrawn
- board text removed: "RESERVED AREA FOR FILTER"
- board text removed: "~"

Commit message: board release candidate
Parts:
- added U$3: (no value), SparkFun-Aesthetics:OSHW-LOGO-L
Routing:
- net SW: track 103.0 -> 101.3 mm
Other:
- outline, holes or cut-outs redrawn
- board text added: "(c)2018 Luca Anastasio"
- board text added: "Lab Access System"
