File: LabAccessBoard/LabAccessBoard.sch (EAGLE design)
At the start: 25 parts, among them CN1 6p-2.54, Q1 AO3400, X1 1751248

Commit message: started firmware development
Parts:
- U$2: value L -> (none); device adafruit:L -> rcl:L-US6000-XXX-RC
Changed lines of the file:
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@@
 <part name="+3V6" library="supply1" library_urn="urn:adsk.eagle:library:371" deviceset="+3V3" device=""/>
 <part name="C5" library="rcl" library_urn="urn:adsk.eagle:library:334" deviceset="C-EU" device="102-064X133" package3d_urn="urn:adsk.eagle:package:23653/1"/>
-<part name="U$2" library="adafruit" library_urn="urn:adsk.eagle:library:420" deviceset="L" device=""/>
+<part name="U$2" library="rcl" library_urn="urn:adsk.eagle:library:334" deviceset="L-US" device="6000-XXX-RC" package3d_urn="urn:adsk.eagle:package:23538/1"/>
 <part name="+3V9" library="supply1" library_urn="urn:adsk.eagle:library:371" deviceset="+3V3" device=""/>
 <part name="C6" library="rcl" library_urn="urn:adsk.eagle:library:334" deviceset="C-EU" device="C0805K" package3d_urn="urn:adsk.eagle:package:23681/2" value="22uF"/>
