File: DoorOpener/DoorOpenerPCB/DoorOpenerPCB.sch (EAGLE design)
At the start: 14 parts, among them IC1 TINY13-20SSU, Q1 AO6602, Q2 AO6602, Q3 2N7002DW

Commit message: pot board
Parts:
- removed C1: (no value), rcl:C-EUC0805K
- removed Q1, Q2: AO6602, SparkFun-DiscreteSemi:MOSFET_COMPLIMENTARY_PAIR-DMC2700UDM
- removed Q3: 2N7002DW, SparkFun-DiscreteSemi:TRANS_NPN_DUAL-MBT3904DW1T1
- added C5: 0.22uF, rcl:C-EUC0603K
- added R4: (no value), rcl:R-TRIMM3103
- added U1: A4950ELJTR-T, allegro:A4950ELJTR-T
- C3: device rcl:C-EUC0805K -> rcl:CPOL-USCT3528
- C4: value (none) -> 0.22uF
- R1: value (none) -> 0.5; device rcl:R-US_R0603 -> rcl:R-US_R0805
Connections:
- new net N$3: R2.1, R4.A
- net +12V: now also C3.+, C5.1, U1.VBB; no longer C1.1, C3.1, Q1.S2, Q2.S2, R1.2, R2.2
- net +5V: now also R2.2
- net GND: now also C3.-, C5.2, R1.1, R4.E, U1.GND, U1.PAD; no longer C1.2, C3.2, Q1.S1, Q2.S1, Q3Q1.E, Q3Q2.E
- net M+: now also U1.OUT1; no longer Q2.D1, Q2.D2
- net M-: now also U1.OUT2; no longer Q1.D1, Q1.D2
- net N$1: now also R4.S, U1.VREF; no longer Q2.G2, Q3Q1.C, R1.1
- net N$2: now also R1.2, U1.LSS; no longer Q1.G2, Q3Q2.C, R2.1
- net PB0: now also U1.IN1; no longer Q2.G1, Q3Q2.B
- net PB1: now also U1.IN2\; no longer Q1.G1, Q3Q1.B
Other:
- moved on the sheet: R1, R2
