File: LabAccess/LabAccessBoard/LabAccessBoard.sch (EAGLE design)
At the start: 25 parts, among them CN1 6p-2.54, Q1 AO3400, X1 1751248

Commit message: board update
Parts:
- removed C4: 100nF, rcl:C-EUC0603K
- removed CN1: 6p-2.54, Seeed-Connector:DIP-BLACK-FEMALE-HEADER-VERT(6P-2.54)
- removed R1, R2, R7: 10k, resistor:R-US_R0603
- added J1: 4p-2.54, Seeed-Connector:DIP-BLACK-MALE-HEADER-VERT(4P-2.54)
Connections:
- removed net EN: C4.2, R7.2, U1.CH_PD
- removed net GPIO0: C4.1, CN1.6, R2.2, U1.GPIO0
- removed net RST: JP1.7, U1.RESET
- new net EXTSW: R6.2, U1.GPIO5, X1-2.K
- net +3V3: now also J1.P$4; no longer CN1.3, R2.1, R7.1
- net CS: now also U1.GPIO16; no longer R1.2, U1.GPIO15
- net GND: now also J1.P$1; no longer CN1.1, R1.1
- net RLY: now also U1.GPIO15; no longer U1.GPIO16
- net RX: now also J1.P$2; no longer CN1.4
- net SW: now also U1.GPIO0; no longer R6.2, U1.GPIO5, X1-2.K
- net TX: now also J1.P$3; no longer CN1.5
Other:
- note added: "INVERTED 4 AND 5 ON MODULE!!!"
- note added: "Internal pull-up/down always 12k: GPIO0 pull-up GPIO15 pull-down RESET pull-up CH_PD pull-up GPIO16 HIGH during boot"
- note added: "built-in LED pull-up not really needed"
- note added: "internal pull-down"
- note added: "internal pull-up"
- moved on the sheet: R3

Commit message: board update
Parts:
- added IC1: TLP281, TLP281(GB-TP_F):TLP281(GB-TP,F)
- added R1: (no value), resistor:R-US_R0603
- added R2, R7: 0, resistor:R-US_R0603
- C5: value (none) -> 100nF
- HLK-PM03: value HLK-PM013W -> HLK-PM03
- R4: value S07K250 -> 250V
- R5: value 2ohm -> 2R
- U$1: value SRD-0XVDC-SL-CSRD-06VDC-SL-C -> SRD-03VDC-SL-C
- U$2: value (none) -> 10mH
- renumbered HLK1 to HLK-PM03
Connections:
- new net A: IC1.ANODE, R2.1, X1-2.K
- new net K: IC1.CATHODE, R1.2, R7.1
- new net K': R1.1, X1-1.K
- net EXTSW: now also IC1.COLLECTOR, R2.2; no longer X1-2.K
- net GND: now also IC1.EMITTER, R7.2; no longer X1-1.K
Other:
- moved on the sheet: R6, X1-1, X1-2

Commit message: board update
Parts:
- removed C3: 100nF, rcl:C-EUC0603K
- C1, C6: value 22uF -> 1uF; device rcl:C-EUC0805K -> rcl:C-EUC0603K
- C2: value 22uF -> 10uF
- D1: value 1N4007 -> 1N4001
- R1: value (none) -> ROC
- R6: value 3.3k -> RSW
Connections:
- removed net K': R1.1, X1-1.K
- new net N$9: R1.1, X1-2.K
- net +3V3: no longer C3.2
- net A: now also R1.2; no longer X1-2.K
- net GND: no longer C3.1
- net K: now also X1-1.K; no longer R1.2
Other:
- moved on the sheet: R1
Changed lines of the file:
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@@
 <setting verticaltext="up"/>
 </settings>
-<grid distance="0.05" unitdist="inch" unit="inch" style="lines" multiple="1" display="no" altdistance="0.01" altunitdist="inch" altunit="inch"/>
+<grid distance="0.1" unitdist="inch" unit="inch" style="lines" multiple="1" display="no" altdistance="0.01" altunitdist="inch" altunit="inch"/>
 <layers>
 <layer number="1" name="Top" color="4" fill="1" visible="no" active="no"/>
@@
 <part name="R5" library="resistor" library_urn="urn:adsk.eagle:library:348" deviceset="R-US_" device="R0603" package3d_urn="urn:adsk.eagle:package:26057/1" value="2R"/>
 <part name="FRAME1" library="SparkFun-Aesthetics" library_urn="urn:adsk.eagle:library:507" deviceset="FRAME-A4L" device=""/>
-<part name="C1" library="rcl" library_urn="urn:adsk.eagle:library:334" deviceset="C-EU" device="C0805K" package3d_urn="urn:adsk.eagle:package:23681/2" value="22uF"/>
-<part name="C2" library="rcl" library_urn="urn:adsk.eagle:library:334" deviceset="C-EU" device="C0805K" package3d_urn="urn:adsk.eagle:package:23681/2" value="22uF"/>
-<part name="C3" library="rcl" library_urn="urn:adsk.eagle:library:334" deviceset="C-EU" device="C0603K" package3d_urn="urn:adsk.eagle:package:23680/2" value="100nF"/>
+<part name="C1" library="rcl" library_urn="urn:adsk.eagle:library:334" deviceset="C-EU" device="C0603K" package3d_urn="urn:adsk.eagle:package:23680/2" value="1uF"/>
+<part name="C2" library="rcl" library_urn="urn:adsk.eagle:library:334" deviceset="C-EU" device="C0805K" package3d_urn="urn:adsk.eagle:package:23681/2" value="10uF"/>
 <part name="Q1" library="Seeed-Transistor" library_urn="urn:adsk.eagle:library:477" deviceset="SMD-MOSFET-N-CH-60V-300MA-LOGIC-LEVEL-FET-2N7002(SOT-23)" device="" package3d_urn="urn:adsk.eagle:package:33015/1" value="AO3400"/>
-<part name="D1" library="Seeed-Diode" library_urn="urn:adsk.eagle:library:467" deviceset="DIODE-GEN-PURPOSE-1KV-1A(DO-214AC)" device="" package3d_urn="urn:adsk.eagle:package:32508/1" value="1N4007"/>
-<part name="R6" library="resistor" library_urn="urn:adsk.eagle:library:348" deviceset="R-US_" device="R0603" package3d_urn="urn:adsk.eagle:package:26057/1" value="3.3k"/>
+<part name="D1" library="Seeed-Diode" library_urn="urn:adsk.eagle:library:467" deviceset="DIODE-GEN-PURPOSE-1KV-1A(DO-214AC)" device="" package3d_urn="urn:adsk.eagle:package:32508/1" value="1N4001"/>
+<part name="R6" library="resistor" library_urn="urn:adsk.eagle:library:348" deviceset="R-US_" device="R0603" package3d_urn="urn:adsk.eagle:package:26057/1" value="RSW"/>
 <part name="R4" library="varistor" library_urn="urn:adsk.eagle:library:410" deviceset="S07K250" device="" package3d_urn="urn:adsk.eagle:package:30540/1" value="250V"/>
 <part name="C5" library="rcl" library_urn="urn:adsk.eagle:library:334" deviceset="C-EU" device="102-064X133" package3d_urn="urn:adsk.eagle:package:23653/1" value="100nF"/>
 <part name="U$2" library="rcl" library_urn="urn:adsk.eagle:library:334" deviceset="L-US" device="6000-XXX-RC" package3d_urn="urn:adsk.eagle:package:23538/1" value="10mH"/>
 <part name="+3V9" library="supply1" library_urn="urn:adsk.eagle:library:371" deviceset="+3V3" device=""/>
-<part name="C6" library="rcl" library_urn="urn:adsk.eagle:library:334" deviceset="C-EU" device="C0805K" package3d_urn="urn:adsk.eagle:package:23681/2" value="22uF"/>
+<part name="C6" library="rcl" library_urn="urn:adsk.eagle:library:334" deviceset="C-EU" device="C0603K" package3d_urn="urn:adsk.eagle:package:23680/2" value="1uF"/>
 <part name="J1" library="Seeed-Connector" library_urn="urn:adsk.eagle:library:478" deviceset="DIP-BLACK-MALE-HEADER-VERT(4P-2.54)" device="" package3d_urn="urn:adsk.eagle:package:33137/1" value="4p-2.54"/>
 <part name="IC1" library="TLP281(GB-TP_F)" deviceset="TLP281(GB-TP,F)" device="" value="TLP281"/>
-<part name="R1" library="resistor" library_urn="urn:adsk.eagle:library:348" deviceset="R-US_" device="R0603" package3d_urn="urn:adsk.eagle:package:26057/1"/>
+<part name="R1" library="resistor" library_urn="urn:adsk.eagle:library:348" deviceset="R-US_" device="R0603" package3d_urn="urn:adsk.eagle:package:26057/1" value="ROC"/>
 <part name="R2" library="resistor" library_urn="urn:adsk.eagle:library:348" deviceset="R-US_" device="R0603" package3d_urn="urn:adsk.eagle:package:26057/1" value="0"/>
 <part name="R7" library="resistor" library_urn="urn:adsk.eagle:library:348" deviceset="R-US_" device="R0603" package3d_urn="urn:adsk.eagle:package:26057/1" value="0"/>
@@
 <instance part="C1" gate="G$1" x="88.9" y="55.88"/>
 <instance part="C2" gate="G$1" x="99.06" y="22.86"/>
-<instance part="C3" gate="G$1" x="111.76" y="22.86"/>
 <instance part="Q1" gate="G$1" x="73.66" y="43.18" rot="MR0"/>
 <instance part="D1" gate="G$1" x="73.66" y="55.88" rot="R90"/>
@@
 <instance part="J1" gate="G$1" x="134.62" y="143.51" rot="R180"/>
 <instance part="IC1" gate="G$1" x="194.31" y="71.12"/>
-<instance part="R1" gate="G$1" x="184.15" y="68.58"/>
+<instance part="R1" gate="G$1" x="184.15" y="71.12"/>
 <instance part="R2" gate="G$1" x="213.36" y="77.47"/>
 <instance part="R7" gate="G$1" x="213.36" y="62.23"/>
@@
 <wire x1="129.54" y1="27.94" x2="121.92" y2="27.94" width="0.1524" layer="91"/>
 <pinref part="C2" gate="G$1" pin="1"/>
-<wire x1="121.92" y1="27.94" x2="111.76" y2="27.94" width="0.1524" layer="91"/>
-<wire x1="111.76" y1="27.94" x2="99.06" y2="27.94" width="0.1524" layer="91"/>
+<wire x1="121.92" y1="27.94" x2="99.06" y2="27.94" width="0.1524" layer="91"/>
 <wire x1="99.06" y1="27.94" x2="91.44" y2="27.94" width="0.1524" layer="91"/>
 <wire x1="99.06" y1="25.4" x2="99.06" y2="27.94" width="0.1524" layer="91"/>
 <junction x="99.06" y="27.94"/>
-<pinref part="C3" gate="G$1" pin="1"/>
-<wire x1="111.76" y1="25.4" x2="111.76" y2="27.94" width="0.1524" layer="91"/>
-<junction x="111.76" y="27.94"/>
 <pinref part="C6" gate="G$1" pin="1"/>
 <wire x1="121.92" y1="25.4" x2="121.92" y2="27.94" width="0.1524" layer="91"/>
@@
 <wire x1="129.54" y1="12.7" x2="121.92" y2="12.7" width="0.1524" layer="91"/>
 <pinref part="C2" gate="G$1" pin="2"/>
-<wire x1="121.92" y1="12.7" x2="111.76" y2="12.7" width="0.1524" layer="91"/>
-<wire x1="111.76" y1="12.7" x2="99.06" y2="12.7" width="0.1524" layer="91"/>
+<wire x1="121.92" y1="12.7" x2="99.06" y2="12.7" width="0.1524" layer="91"/>
 <wire x1="99.06" y1="12.7" x2="91.44" y2="12.7" width="0.1524" layer="91"/>
 <wire x1="99.06" y1="17.78" x2="99.06" y2="12.7" width="0.1524" layer="91"/>
 <junction x="99.06" y="12.7"/>
-<pinref part="C3" gate="G$1" pin="2"/>
-<wire x1="111.76" y1="17.78" x2="111.76" y2="12.7" width="0.1524" layer="91"/>
-<junction x="111.76" y="12.7"/>
 <pinref part="C6" gate="G$1" pin="2"/>
 <wire x1="121.92" y1="17.78" x2="121.92" y2="12.7" width="0.1524" layer="91"/>
@@
 <wire x1="191.77" y1="71.12" x2="191.77" y2="77.47" width="0.1524" layer="91"/>
 <wire x1="191.77" y1="77.47" x2="208.28" y2="77.47" width="0.1524" layer="91"/>
-<pinref part="X1" gate="-2" pin="K"/>
-<wire x1="176.53" y1="71.12" x2="191.77" y2="71.12" width="0.1524" layer="91"/>
-<junction x="191.77" y="71.12"/>
-<label x="176.53" y="71.12" size="1.778" layer="95"/>
-</segment>
-</net>
-<net name="K'" class="0">
-<segment>
-<pinref part="X1" gate="-1" pin="K"/>
-<pinref part="R1" gate="G$1" pin="1"/>
-<wire x1="176.53" y1="68.58" x2="179.07" y2="68.58" width="0.1524" layer="91"/>
-<label x="176.53" y="68.58" size="1.778" layer="95"/>
+<pinref part="R1" gate="G$1" pin="2"/>
+<wire x1="189.23" y1="71.12" x2="194.31" y2="71.12" width="0.1524" layer="91"/>
+<junction x="194.31" y="71.12"/>
+<label x="190.5" y="71.12" size="1.778" layer="95"/>
 </segment>
 </net>
@@
 <segment>
 <pinref part="IC1" gate="G$1" pin="CATHODE"/>
-<label x="191.77" y="68.58" size="1.778" layer="95"/>
 <pinref part="R7" gate="G$1" pin="1"/>
 <wire x1="191.77" y1="68.58" x2="194.31" y2="68.58" width="0.1524" layer="91"/>
 <wire x1="191.77" y1="68.58" x2="191.77" y2="62.23" width="0.1524" layer="91"/>
 <wire x1="191.77" y1="62.23" x2="208.28" y2="62.23" width="0.1524" layer="91"/>
-<pinref part="R1" gate="G$1" pin="2"/>
-<wire x1="189.23" y1="68.58" x2="191.77" y2="68.58" width="0.1524" layer="91"/>
-<junction x="191.77" y="68.58"/>
-</segment>
-</net>
+<pinref part="X1" gate="-1" pin="K"/>
+<wire x1="176.53" y1="68.58" x2="194.31" y2="68.58" width="0.1524" layer="91"/>
+<junction x="194.31" y="68.58"/>
+<label x="190.5" y="68.58" size="1.778" layer="95"/>
+</segment>
+</net>
+<net name="N$9" class="0">
+<segment>
+<pinref part="X1" gate="-2" pin="K"/>
+<pinref part="R1" gate="G$1" pin="1"/>
+<wire x1="176.53" y1="71.12" x2="179.07" y2="71.12" width="0.1524" layer="91"/>
+</segment>
+</net>

Commit message: new lab access board
Parts:
- removed D1: 1N4001, Seeed-Diode:DIODE-GEN-PURPOSE-1KV-1A(DO-214AC)
- added D2: 250mA/100V, SparkFun-DiscreteSemi:DIODE-BAS16J
Connections:
- net N$5: now also D2.C; no longer D1.-
- net N$8: now also D2.A; no longer D1.+
